File: schematic/Theremin.kicad_sch (KiCad schematic)
At the start: 56 parts, among them Q1 2N7002, Q10 BC817, Q2 2N7002, Q3 2N7002, Q4 BC817, Q5 BC817, Q6 2N7002, Q7 2N7002, Q8 2N7002, Q9 BC817, U1 NE555D, U2 AZV3002, U3 MAX4392, U4 MAX4392, U5 NE555D, U6 AZV3002

Commit message: Continued schematic
Parts:
- removed Q1, Q2, Q3, Q6, Q7, Q8: 2N7002, Package_TO_SOT_SMD:SOT-23, symbol Transistor_FET:2N7002
- removed Q10, Q4, Q5, Q9: BC817, Package_TO_SOT_SMD:SOT-23, symbol Transistor_BJT:BC817
- removed TP1, TP2, TP3, TP4, TP5, TP6, TP7, TP8: TestPoint, TestPoint:TestPoint_Pad_D1.5mm, symbol Connector:TestPoint
- removed U4: MAX4392, Package_SO:SOIC-8_3.9x4.9mm_P1.27mm, symbol Device:Opamp_Dual
- removed U5: NE555D, Package_SO:SOIC-8_3.9x4.9mm_P1.27mm, symbol Timer:NE555D
- removed U6: AZV3002, Package_SO:SOIC-8_3.9x4.9mm_P1.27mm, symbol Device:Opamp_Dual
- added Q1, Q2, Q3, Q4, Q5, Q6, Q7, Q8: 2N7000, Package_TO_SOT_THT:TO-92_Inline, symbol Transistor_FET:2N7000
- added R21: ?, Resistor_SMD:R_0805_2012Metric, symbol Device:R
- added R22, R23, R24: 100k, Resistor_SMD:R_0805_2012Metric, symbol Device:R
- added RV1, RV2: 10k, symbol Device:R_Potentiometer
- added U4: NE555D, Package_SO:SOIC-8_3.9x4.9mm_P1.27mm, symbol Timer:NE555D
- added U5: AZV3002, Package_SO:SOIC-8_3.9x4.9mm_P1.27mm, symbol Device:Opamp_Dual
- added U7: Pico, RPi_Pico:RPi_Pico_SMD_TH, symbol Pico:Pico
- C10, C3, C4, C9: value 10n -> ?
- R11, R15, R5: value 220 -> ?
- R12, R6: value 10k -> ?
- R13: value 100k -> 220
- R14: value 1M -> 10k
- R16: value 10k -> 100k
- R17: value 22k -> 1M
- R18, R19, R20: value 100k -> ?
- R7: value 22k -> ?
Connections:
- net +5V: now also R11.1, R14.1, R15.1, R20.1, R6.1, R22.2, R24.2, U4.4 (R), U4.8 (VCC), U5.8 (V+); no longer R12.1, R17.1, R18.2, R20.2, R7.1
- net GND: now also R12.2, R18.2, Q1.1 (S), Q2.1 (S), Q3.1 (S), Q4.1 (S), Q5.1 (S), Q6.1 (S), Q7.1 (S), Q8.1 (S), R23.1, U4.1 (GND), U5.4 (V-); no longer R19.1
- net at C9.1: now also R19.2, Q7.2 (G); no longer R14.2
- net at R13.2: now also C7.1, U4.6 (THR); no longer R14.1
- net at R1.1, U1.3 (Q): now also Q1.2 (G), Q2.2 (G)
- net at R11.2: now also RV1.1; no longer C7.1
- net at R15.2: now also RV2.1; no longer R16.1
- net at R16.2: now also R17.1, U5.3 (+)
- net at R4.2, U2.1: now also R5.1; no longer C3.1, U3.5 (+)
- net ShieldV: now reaches U3.6 (-)
- net ShieldV: now also U3.7; no longer R5.1
- net at R6.2: now also Q3.3 (D), Q4.2 (G)
- net DisM renamed DisMF
- net DisMF: now also Q1.3 (D); no longer C12.1, R20.1
- net DisR renamed DisRF
- net DisRF: now also Q2.3 (D); no longer C8.1, R12.2, R13.1
- net Feedback: no longer names the net of U2.2 (-)
- net Feedback: now also RV1.2
- net Output renamed OutFreq
- net OutFreq: now also Q4.3 (D); no longer C10.1, R17.2
- net RaceEnd renamed RaceEndFreq
- net Shield renamed ShieldF
- new net: R17.2, R19.1, U5.1
- new net: RV2.2, U5.2 (-)
- new net: Q5.2 (G), Q6.2 (G), R13.1, U4.3 (Q)
- new net: R12.1, RV1.3
- new net: C3.1, Q3.2 (G), R5.2
- new net: C11.1, R22.1, R23.2, U5.5 (+)
- new net: R18.1, RV2.3
- new net: Q7.3 (D), Q8.2 (G), R20.2
- new net +3V3: R21.1, R7.1
- new net DisMV: C12.1, Q6.3 (D), R24.1, U3.5 (+), U5.6 (-)
- new net DisRV: C8.1, Q5.3 (D), R14.2, R16.1
- new net OutVol: C10.1, Q8.3 (D), R21.2
- new net RaceEndVol: U4.2 (TR), U5.7
Other:
- moved on the sheet: C1, C2, C3, C4, C5, C6, R1, R10, R2, R3, R4, R7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

Commit message: SCHEMATIC : continued schematic
Parts:
- added D1, D10, D11, D12, D2, D3, D4, D5, D6, D7, D8, D9: ~, symbol Device:D
- added D13, D14, D15, D16, D17, D18, D19, D20, D21, D22, D23, D24: ~, symbol Device:LED_45deg
- added RV3: 10k, symbol Device:R_Potentiometer
- added SW1, SW10, SW11, SW12, SW2, SW3, SW4, SW5, SW6, SW7, SW8, SW9: ~, symbol Switch:SW_Push_45deg
Connections:
- net +3V3: now also RV3.3
- net GND: now also U7.13 (GND), U7.18 (GND), U7.23 (GND), U7.28 (GND), U7.3 (GND), U7.33 (AGND), U7.38 (GND), U7.8 (GND), RV3.1
- net OutFreq: now also U7.31 (GPIO26_ADC0)
- net OutVol: now also U7.32 (GPIO27_ADC1)
- net Echo: now reaches U7.34 (GPIO28_ADC2)
- net Echo: now also RV3.2
- new net: D2.2 (A), SW2.2
- new net: D1.2 (A), SW1.2
- new net: D8.2 (A), SW8.2
- new net: D11.2 (A), SW11.2
- new net: D6.2 (A), SW6.2
- new net: D10.2 (A), SW10.2
- new net: D3.2 (A), SW3.2
- new net: D9.2 (A), SW9.2
- new net: D7.2 (A), SW7.2
- new net: D5.2 (A), SW5.2
- new net: D4.2 (A), SW4.2
- new net: D12.2 (A), SW12.2
- new net LMC0: D13.1 (K), D16.1 (K), D19.1 (K), D20.1 (K)
- new net LMC1: D14.1 (K), D17.1 (K), D21.1 (K), D22.1 (K)
- new net LMC2: D15.1 (K), D18.1 (K), D23.1 (K), D24.1 (K)
- new net LMR0: D13.2 (A), D14.2 (A), D15.2 (A)
- new net LMR1: D16.2 (A), D17.2 (A), D18.2 (A)
- new net LMR2: D19.2 (A), D21.2 (A), D23.2 (A)
- new net LMR3: D20.2 (A), D22.2 (A), D24.2 (A)
- new net SMC0: D1.1 (K), D10.1 (K), D4.1 (K), D7.1 (K)
- new net SMC1: D11.1 (K), D2.1 (K), D5.1 (K), D8.1 (K)
- new net SMC2: D12.1 (K), D3.1 (K), D6.1 (K), D9.1 (K)
- new net SMR0: SW1.1, SW2.1, SW3.1
- new net SMR1: SW4.1, SW5.1, SW6.1
- new net SMR2: SW7.1, SW8.1, SW9.1
- new net SMR3: SW10.1, SW11.1, SW12.1

Commit message: code + schematic + models??
Parts:
- removed C1, C7, C8: 1n, Capacitor_SMD:C_0805_2012Metric, symbol Device:C
- removed C10, C9: ?, Capacitor_SMD:C_0805_2012Metric, symbol Device:C
- removed C11: 100n, Capacitor_SMD:C_0805_2012Metric, symbol Device:C
- removed C12: 20p, Capacitor_SMD:C_0805_2012Metric, symbol Device:C
- removed Q5, Q6, Q7, Q8: 2N7000, Package_TO_SOT_THT:TO-92_Inline, symbol Transistor_FET:2N7000
- removed R13: 220, Resistor_SMD:R_0805_2012Metric, symbol Device:R
- removed R14: 10k, Resistor_SMD:R_0805_2012Metric, symbol Device:R
- removed R15, R18, R19, R20, R21, R5: ?, Resistor_SMD:R_0805_2012Metric, symbol Device:R
- removed R16, R22, R23, R24: 100k, Resistor_SMD:R_0805_2012Metric, symbol Device:R
- removed R17: 1M, Resistor_SMD:R_0805_2012Metric, symbol Device:R
- removed RV2: 10k, symbol Device:R_Potentiometer
- removed unit 2 of U3
- removed U4: NE555D, Package_SO:SOIC-8_3.9x4.9mm_P1.27mm, symbol Timer:NE555D
- removed U5: AZV3002, Package_SO:SOIC-8_3.9x4.9mm_P1.27mm, symbol Device:Opamp_Dual
- C2, C5, C6: footprint Capacitor_SMD:C_0805_2012Metric -> Capacitor_THT:C_Disc_D4.3mm_W1.9mm_P5.00mm
- C3: value ? -> 1n; footprint Capacitor_SMD:C_0805_2012Metric -> Capacitor_THT:C_Disc_D4.3mm_W1.9mm_P5.00mm
- C4: value ? -> 1u; footprint Capacitor_SMD:C_0805_2012Metric -> Capacitor_THT:C_Disc_D4.3mm_W1.9mm_P5.00mm
- Q1, Q2, Q3, Q4: footprint Package_TO_SOT_THT:TO-92_Inline -> Package_TO_SOT_THT:TO-92_Inline_Wide
- R1, R10, R11, R12, R2, R3, R4, R8, R9: footprint Resistor_SMD:R_0805_2012Metric -> Resistor_THT:R_Axial_DIN0207_L6.3mm_D2.5mm_P10.16mm_Horizontal
- R6: value ? -> 100k; footprint Resistor_SMD:R_0805_2012Metric -> Resistor_THT:R_Axial_DIN0207_L6.3mm_D2.5mm_P10.16mm_Horizontal
- R7: value ? -> 56k; footprint Resistor_SMD:R_0805_2012Metric -> Resistor_THT:R_Axial_DIN0207_L6.3mm_D2.5mm_P10.16mm_Horizontal
- U1, U2, U3: footprint Package_SO:SOIC-8_3.9x4.9mm_P1.27mm -> Package_DIP:DIP-8_W7.62mm
Connections:
- net +5V: now also Q4.3 (D); no longer R6.1
- net GND: now also R6.2; no longer Q4.1 (S)
- net OutFreq: now also Q3.3 (D); no longer Q4.3 (D)
- net at R4.2, U2.1: now also C3.1, Q4.2 (G)
- net at Q3.2 (G): now also Q4.1 (S), R6.1; no longer C3.1
- no-connect marks 4 -> 2
Other:
- moved on the sheet: Q3, Q4, R6, U3C
